File: charger.brd (EAGLE design)
At the start: 34 x 24.1 mm, 15 parts, among them IC1 LM317, IC2 LM3420AM5X-8.4

Commit message: minor update
Parts:
- D1: value 1N4004 -> 1N4001
Connections:
- net N$4 renamed V+
Changed lines of the file:
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@@
 <attribute name="VALUE" x="13.335" y="0.635" size="1.27" layer="27"/>
 </element>
-<element name="D1" library="diode" package="DO41-10" value="1N4004" x="21.59" y="10.16" rot="R180"/>
+<element name="D1" library="diode" package="DO41-10" value="1N4001" x="21.59" y="10.16" rot="R180"/>
 <element name="IC1" library="v-reg" package="317TS" value="LM317" x="16.51" y="20.32" smashed="yes">
 <attribute name="NAME" x="11.43" y="14.2748" size="1.27" layer="25" ratio="10"/>
@@
 <wire x1="5.08" y1="8.89" x2="8.89" y2="7.62" width="1.016" layer="16"/>
 </signal>
-<signal name="N$4">
+<signal name="V+">
 <contactref element="IC1" pad="3"/>
 <contactref element="R5" pad="1"/>

Commit message: minor layout fix
Routing:
- net N$7: track 18.0 -> 8.88 mm
- net N$5: track 17.1 -> 12.8 mm
Changed lines of the file:
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@@
 <layers>
 <layer number="1" name="Top" color="4" fill="1" visible="yes" active="yes"/>
-<layer number="16" name="Bottom" color="1" fill="1" visible="yes" active="yes"/>
+<layer number="16" name="Bottom" color="1" fill="1" visible="no" active="yes"/>
 <layer number="17" name="Pads" color="2" fill="1" visible="yes" active="yes"/>
 <layer number="18" name="Vias" color="2" fill="1" visible="yes" active="yes"/>
@@
 <element name="Q1" library="custom" package="TO92" value="" x="5.08" y="7.62" rot="R90"/>
 <element name="Q2" library="custom" package="TO92" value="" x="21.59" y="3.81" smashed="yes" rot="R270">
-<attribute name="NAME" x="18.415" y="4.445" size="1.27" layer="25" ratio="10" rot="R270"/>
+<attribute name="NAME" x="24.765" y="3.175" size="1.27" layer="25" ratio="10" rot="R270"/>
 <attribute name="VALUE" x="20.32" y="0.635" size="1.27" layer="27" ratio="10" rot="R270"/>
 </element>
@@
 <element name="R2" library="rcl" package="0204V" value="1k" x="10.16" y="7.62" smashed="yes">
 <attribute name="NAME" x="8.0264" y="8.7884" size="1.27" layer="25" ratio="10"/>
-<attribute name="VALUE" x="9.2964" y="5.3086" size="1.27" layer="27" ratio="10"/>
-</element>
-<element name="R3" library="rcl" package="0204V" value="100k" x="11.43" y="3.81" rot="R270"/>
+<attribute name="VALUE" x="6.7564" y="10.3886" size="1.27" layer="27" ratio="10"/>
+</element>
+<element name="R3" library="rcl" package="0204V" value="100k" x="11.43" y="3.81" smashed="yes" rot="R270">
+<attribute name="NAME" x="12.5984" y="3.4036" size="1.27" layer="25" ratio="10" rot="R270"/>
+<attribute name="VALUE" x="10.3886" y="0.8636" size="1.27" layer="27" ratio="10" rot="R270"/>
+</element>
 <element name="R4" library="rcl" package="0204V" value="1k" x="8.89" y="3.81" smashed="yes" rot="R90">
-<attribute name="NAME" x="10.2616" y="0.4064" size="1.27" layer="25" ratio="10" rot="R90"/>
-<attribute name="VALUE" x="8.6614" y="0.4064" size="1.27" layer="27" ratio="10" rot="R90"/>
+<attribute name="NAME" x="5.1816" y="0.4064" size="1.27" layer="25" ratio="10" rot="R90"/>
+<attribute name="VALUE" x="7.3914" y="0.4064" size="1.27" layer="27" ratio="10" rot="R90"/>
 </element>
 <element name="R5" library="rcl" package="0204V" value="10k" x="25.4" y="12.7" smashed="yes" rot="R180">
@@
 <wire x1="25.6032" y1="7.5438" x2="25.82" y2="7.62" width="0.254" layer="16"/>
 <wire x1="26.5176" y1="12.573" x2="26.67" y2="12.7" width="0.254" layer="16"/>
-<wire x1="27.6606" y1="12.573" x2="26.7462" y2="12.573" width="0.254" layer="1"/>
-<wire x1="28.8036" y1="11.43" x2="27.6606" y2="12.573" width="0.254" layer="1"/>
-<wire x1="30.48" y1="11.43" x2="28.8036" y2="11.43" width="0.254" layer="1"/>
+<wire x1="27.6606" y1="12.573" x2="26.7462" y2="12.573" width="1.016" layer="1"/>
+<wire x1="28.8036" y1="11.43" x2="27.6606" y2="12.573" width="1.016" layer="1"/>
+<wire x1="30.48" y1="11.43" x2="28.8036" y2="11.43" width="1.016" layer="1"/>
 <wire x1="26.7462" y1="12.573" x2="26.67" y2="12.7" width="0.254" layer="1"/>
 </signal>
@@
 <wire x1="16.2306" y1="4.572" x2="16.2306" y2="5.0292" width="0.254" layer="1"/>
 <wire x1="16.2306" y1="5.0292" x2="16.19" y2="5.044" width="0.254" layer="1"/>
-<wire x1="5.2578" y1="2.7432" x2="8.89" y2="5.08" width="0.254" layer="16"/>
 <wire x1="16.2306" y1="4.572" x2="16.09" y2="4.572" width="0.4064" layer="1"/>
 <wire x1="16.09" y1="4.572" x2="16.09" y2="2.54" width="0.4064" layer="1"/>
@@
 <contactref element="R4" pad="1"/>
 <contactref element="Q1" pad="2"/>
-<wire x1="2.7432" y1="2.7432" x2="8.89" y2="2.54" width="0.254" layer="16"/>
-<wire x1="2.0574" y1="3.2004" x2="2.0574" y2="6.1722" width="0.254" layer="16"/>
-<wire x1="2.5146" y1="2.7432" x2="2.0574" y2="3.2004" width="0.254" layer="16"/>
-<wire x1="2.0574" y1="6.1722" x2="3.175" y2="7.62" width="0.254" layer="16"/>
-<wire x1="2.5146" y1="2.7432" x2="8.89" y2="2.54" width="0.254" layer="16"/>
+<wire x1="3.048" y1="6.5532" x2="3.048" y2="7.62" width="0.1524" layer="1"/>
+<wire x1="3.5052" y1="6.096" x2="3.048" y2="6.5532" width="0.1524" layer="1"/>
+<wire x1="3.5052" y1="5.7912" x2="3.5052" y2="6.096" width="0.1524" layer="1"/>
+<wire x1="6.7056" y1="2.5908" x2="3.5052" y2="5.7912" width="0.1524" layer="1"/>
+<wire x1="8.8392" y1="2.5908" x2="6.7056" y2="2.5908" width="0.1524" layer="1"/>
+<wire x1="3.048" y1="7.62" x2="3.175" y2="7.62" width="0.1524" layer="1"/>
+<wire x1="8.8392" y1="2.5908" x2="8.89" y2="2.54" width="0.1524" layer="1"/>
 </signal>
 <signal name="N$8">
